Commit message: Copied urdf I was using before from a different package.

File: src/baxter.urdf (robot description, URDF)
Before this commit: robot baxter, 53 links, 52 joints
Links:
- added link block, mass 0.0001; collision box size=0.05 0.05 0.05; visual box size=0.05 0.05 0.05
- link left_gripper_left: geometry collision box size=0.02 0.01 0.1; visual box size=0.02 0.01 0.1
- link left_gripper_right: geometry collision box size=0.02 0.01 0.1; visual box size=0.02 0.01 0.1
- link right_gripper_left: geometry collision box size=0.02 0.01 0.1; visual box size=0.02 0.01 0.1
- link right_gripper_right: geometry collision box size=0.02 0.01 0.1; visual box size=0.02 0.01 0.1
Joints:
- added joint block: type fixed, parent left_gripper, child block, origin xyz=0.0 0.0 0.05 rpy=0 0 0

Commit message: Removed block and went back to using as a collision object, still modified from original for grippers. Disabled few links in collision with display that should not be considered.

File: src/baxter.urdf (robot description, URDF)
Before this commit: robot baxter, 54 links, 53 joints
Links:
- removed link block
Joints:
- removed joint block
